Commit message: set xacro for gazebo spawn

File: trip_description/urdf/trip.urdf.xacro (robot description, xacro)
@@ -1,25 +1,195 @@
 <?xml version="1.0"?>
-<robot xmlns:xacro="http://www.ros.org/wiki/xacro" name="trip">
-    <material name="grey">
-        <color rgba="0.7 0.7 0.7 1.0"/>
-    </material>
-    <!-- Base link -->
-    <link name="base_link">
-        <inertial>
-            <origin xyz="0 0 0" rpy="0 0 0"/>
-            <mass value="1.0"/>
-            <inertia
-                ixx="0.01" ixy="0.0" ixz="0.0"
-                iyy="0.01" iyz="0.0"
-                izz="0.01"/>
-        </inertial>
-        <visual>
-            <!-- <origin xyz="-0.02 0.11 0" rpy="0 0 3.14"/> -->
-            <origin xyz="0 0 0" rpy="0 0 0"/>
-            <geometry>
-                <mesh filename="package://trip_description/meshes/base_link.stl" scale="1 1 1"/>
-            </geometry>
-            <material name="grey"/>
-        </visual>
+<robot name="trip" xmlns:xacro="http://www.ros.org/wiki/xacro">
+  <xacro:property name="pi" value="3.141592653589793"/>
+  <!--  BASE LINK  -->
+  <link name="base_link">
+    <inertial>
+      <origin xyz="0 0 0" rpy="0 0 0"/>
+      <mass value="5.0"/>
+      <inertia
+        ixx="0.05" ixy="0.0" ixz="0.0"
+        iyy="0.05" iyz="0.0"
+        izz="0.08"/>
+    </inertial>
+    <visual>
+      <origin xyz="0.003 -0.002 -0.075" rpy="0 0 ${pi}"/>
+      <geometry>
+          <mesh filename="package://trip_description/meshes/base_link.dae"/>
+      </geometry>
+    </visual>
+    <collision>
+      <origin xyz="-0.004 0 0" rpy="0 0 0"/>
+      <geometry>
+        <box size="0.16 0.103 0.11"/>
+      </geometry>
+    </collision>
+  </link>
+  <!--  IMU  -->
+  <link name="imu_link">
+    <inertial>
+      <mass value="0.01"/>
+      <inertia
+        ixx="1e-5" ixy="0.0" ixz="0.0"
+        iyy="1e-5" iyz="0.0"
+        izz="1e-5"/>
+    </inertial>
+  </link>
+  <joint name="imu_joint" type="fixed">
+    <parent link="base_link"/>
+    <child link="imu_link"/>
+    <origin xyz="0 0 0.08" rpy="0 0 0"/>
+  </joint>
+  <gazebo reference="imu_link">
+    <sensor name="imu_sensor" type="imu">
+      <always_on>true</always_on>
+      <update_rate>200</update_rate>
+      <imu>
+        <angular_velocity>
+          <x><noise type="gaussian"><stddev>0.002</stddev></noise></x>
+          <y><noise type="gaussian"><stddev>0.002</stddev></noise></y>
+          <z><noise type="gaussian"><stddev>0.002</stddev></noise></z>
+        </angular_velocity>
+        <linear_acceleration>
+          <x><noise type="gaussian"><stddev>0.03</stddev></noise></x>
+          <y><noise type="gaussian"><stddev>0.03</stddev></noise></y>
+          <z><noise type="gaussian"><stddev>0.03</stddev></noise></z>
+        </linear_acceleration>
+      </imu>
+      <plugin name="imu_plugin" filename="libgazebo_ros_imu_sensor.so">
+        <ros>
+          <namespace>/trip</namespace>
+          <remapping>~/out:=imu</remapping>
+        </ros>
+        <frame_name>imu_link</frame_name>
+      </plugin>
+    </sensor>
+  </gazebo>
+  <!--  CAMERA  -->
+  <link name="camera_link">
+    <inertial>
+      <mass value="0.01"/>
+      <inertia
+        ixx="1e-5" ixy="0.0" ixz="0.0"
+        iyy="1e-5" iyz="0.0"
+        izz="1e-5"/>
+    </inertial>
+  </link>
+  <joint name="camera_joint" type="fixed">
+    <parent link="base_link"/>
+    <child link="camera_link"/>
+    <origin xyz="0.08 0 0.12" rpy="0 0 0"/>
+  </joint>
+  <gazebo reference="camera_link">
+    <sensor name="camera_sensor" type="camera">
+      <update_rate>30</update_rate>
+      <camera>
+        <horizontal_fov>1.396</horizontal_fov>
+        <image>
+          <width>640</width>
+          <height>480</height>
+          <format>R8G8B8</format>
+        </image>
+        <clip><near>0.05</near><far>50</far></clip>
+      </camera>
+      <plugin name="trip_camera_plugin" filename="libgazebo_ros_camera.so">
+        <ros><namespace>/trip</namespace></ros>
+        <frame_name>camera_link</frame_name>
+        <camera_name>camera</camera_name>
+        <image_topic_name>image_raw</image_topic_name>
+        <camera_info_topic_name>camera_info</camera_info_topic_name>
+      </plugin>
+    </sensor>
+  </gazebo>
+  <!--  LIDAR  -->
+  <link name="lidar_pitch_link">
+    <visual>
+      <geometry>
+        <box size="0.04 0.04 0.01"/>
+      </geometry>
+    </visual>
+    <inertial>
+      <mass value="0.1"/>
+      <inertia ixx="0.0005" iyy="0.0005" izz="0.0005"
+              ixy="0" ixz="0" iyz="0"/>
+    </inertial>
+  </link>
+  <link name="lidar_link">
+    <visual>
+      <geometry>
+        <cylinder radius="0.015" length="0.02"/>
+      </geometry>
+    </visual>
+    <inertial>
+      <mass value="0.01"/>
+      <inertia
+        ixx="1e-5" ixy="0.0" ixz="0.0"
+        iyy="1e-5" iyz="0.0"
+        izz="1e-5"/>
+    </inertial>
+  </link>
+  <joint name="lidar_pitch_joint" type="revolute">
+    <parent link="base_link"/>
+    <child link="lidar_pitch_link"/>
+    <origin xyz="0.04 0 0.09" rpy="0 0 0"/>
+    <axis xyz="1 0 0"/>
+    <limit lower="-0.35" upper="0.35" effort="1.0" velocity="1.0"/>
+  </joint>
+  <joint name="lidar_mount_joint" type="fixed">
+    <parent link="lidar_pitch_link"/>
+    <child link="lidar_link"/>
+    <origin xyz="0 0 0.01" rpy="0 0 0"/>
+  </joint>
+  <gazebo reference="lidar_link">
+    <sensor name="lidar_sensor" type="ray">
+      <update_rate>10</update_rate>
+      <ray>
+        <scan>
+          <horizontal>
+            <samples>720</samples>
+            <min_angle>-1.5708</min_angle>
+            <max_angle>1.5708</max_angle>
+          </horizontal>
+        </scan>
+        <range>
+          <min>0.12</min>
+          <max>30.0</max>
+          <resolution>0.01</resolution>
+        </range>
+      </ray>
+      <plugin name="trip_lidar_plugin" filename="libgazebo_ros_ray_sensor.so">
+        <ros>
+          <namespace>/trip</namespace>
+          <remapping>~/out:=scan</remapping>
+        </ros>
+        <frame_name>lidar_link</frame_name>
+        <output_type>sensor_msgs/LaserScan</output_type>
+      </plugin>
+    </sensor>
+  </gazebo>
+  <xacro:macro name="wheel" params="name x y">
+    <link name="${name}">
+      <collision>
+        <geometry>
+          <cylinder radius="0.034" length="0.027"/>
+        </geometry>
+      </collision>
+      <inertial>
+        <mass value="0.1"/>
+        <inertia
+          ixx="1e-4" ixy="0" ixz="0"
+          iyy="1e-4" iyz="0"
+          izz="1e-4"/>
+      </inertial>
     </link>
+    <joint name="${name}_joint" type="continuous">
+      <parent link="base_link"/>
+      <child link="${name}"/>
+      <origin xyz="${x} ${y} -0.042" rpy="0 ${pi/2} ${pi/2}"/>
+      <axis xyz="0 0 1"/>
+    </joint>
+  </xacro:macro>
+  <xacro:wheel name="right_front_wheel" x="0.07"  y="-0.0716"/>
+  <xacro:wheel name="left_front_wheel"  x="0.07"  y="0.0716"/>
+  <xacro:wheel name="right_back_wheel"  x="-0.07" y="-0.0716"/>
+  <xacro:wheel name="left_back_wheel"   x="-0.07" y="0.0716"/>
 </robot>

Commit message: fix absolute path and minor changes

File: trip_description/urdf/trip.urdf.xacro (robot description, xacro)
@@ -2,4 +2,7 @@
 <robot name="trip" xmlns:xacro="http://www.ros.org/wiki/xacro">
   <xacro:property name="pi" value="3.141592653589793"/>
+  <material name="light_black">
+    <color rgba="0.4 0.4 0.4 1.0"/>
+  </material>
   <!--  BASE LINK  -->
   <link name="base_link">
@@ -15,6 +18,7 @@
       <origin xyz="0.003 -0.002 -0.075" rpy="0 0 ${pi}"/>
       <geometry>
-          <mesh filename="package://trip_description/meshes/base_link.dae"/>
+          <mesh filename="/home/davdori/trip_ws/src/TRIP-sim/trip_description/meshes/base_link.dae"/>
       </geometry>
+      <material name="light_black"/>
     </visual>
     <collision>

Commit message: split main xacro in submodules

File: trip_description/urdf/trip.urdf.xacro (robot description, xacro)
@@ -1,199 +1,15 @@
 <?xml version="1.0"?>
 <robot name="trip" xmlns:xacro="http://www.ros.org/wiki/xacro">
-  <xacro:property name="pi" value="3.141592653589793"/>
-  <material name="light_black">
-    <color rgba="0.4 0.4 0.4 1.0"/>
-  </material>
-  <!--  BASE LINK  -->
-  <link name="base_link">
-    <inertial>
-      <origin xyz="0 0 0" rpy="0 0 0"/>
-      <mass value="5.0"/>
-      <inertia
-        ixx="0.05" ixy="0.0" ixz="0.0"
-        iyy="0.05" iyz="0.0"
-        izz="0.08"/>
-    </inertial>
-    <visual>
-      <origin xyz="0.003 -0.002 -0.075" rpy="0 0 ${pi}"/>
-      <geometry>
-          <mesh filename="/home/davdori/trip_ws/src/TRIP-sim/trip_description/meshes/base_link.dae"/>
-      </geometry>
-      <material name="light_black"/>
-    </visual>
-    <collision>
-      <origin xyz="-0.004 0 0" rpy="0 0 0"/>
-      <geometry>
-        <box size="0.16 0.103 0.11"/>
-      </geometry>
-    </collision>
-  </link>
-  <!--  IMU  -->
-  <link name="imu_link">
-    <inertial>
-      <mass value="0.01"/>
-      <inertia
-        ixx="1e-5" ixy="0.0" ixz="0.0"
-        iyy="1e-5" iyz="0.0"
-        izz="1e-5"/>
-    </inertial>
-  </link>
-  <joint name="imu_joint" type="fixed">
-    <parent link="base_link"/>
-    <child link="imu_link"/>
-    <origin xyz="0 0 0.08" rpy="0 0 0"/>
-  </joint>
-  <gazebo reference="imu_link">
-    <sensor name="imu_sensor" type="imu">
-      <always_on>true</always_on>
-      <update_rate>200</update_rate>
-      <imu>
-        <angular_velocity>
-          <x><noise type="gaussian"><stddev>0.002</stddev></noise></x>
-          <y><noise type="gaussian"><stddev>0.002</stddev></noise></y>
-          <z><noise type="gaussian"><stddev>0.002</stddev></noise></z>
-        </angular_velocity>
-        <linear_acceleration>
-          <x><noise type="gaussian"><stddev>0.03</stddev></noise></x>
-          <y><noise type="gaussian"><stddev>0.03</stddev></noise></y>
-          <z><noise type="gaussian"><stddev>0.03</stddev></noise></z>
-        </linear_acceleration>
-      </imu>
-      <plugin name="imu_plugin" filename="libgazebo_ros_imu_sensor.so">
-        <ros>
-          <namespace>/trip</namespace>
-          <remapping>~/out:=imu</remapping>
-        </ros>
-        <frame_name>imu_link</frame_name>
-      </plugin>
-    </sensor>
-  </gazebo>
-  <!--  CAMERA  -->
-  <link name="camera_link">
-    <inertial>
-      <mass value="0.01"/>
-      <inertia
-        ixx="1e-5" ixy="0.0" ixz="0.0"
-        iyy="1e-5" iyz="0.0"
-        izz="1e-5"/>
-    </inertial>
-  </link>
-  <joint name="camera_joint" type="fixed">
-    <parent link="base_link"/>
-    <child link="camera_link"/>
-    <origin xyz="0.08 0 0.12" rpy="0 0 0"/>
-  </joint>
-  <gazebo reference="camera_link">
-    <sensor name="camera_sensor" type="camera">
-      <update_rate>30</update_rate>
-      <camera>
-        <horizontal_fov>1.396</horizontal_fov>
-        <image>
-          <width>640</width>
-          <height>480</height>
-          <format>R8G8B8</format>
-        </image>
-        <clip><near>0.05</near><far>50</far></clip>
-      </camera>
-      <plugin name="trip_camera_plugin" filename="libgazebo_ros_camera.so">
-        <ros><namespace>/trip</namespace></ros>
-        <frame_name>camera_link</frame_name>
-        <camera_name>camera</camera_name>
-        <image_topic_name>image_raw</image_topic_name>
-        <camera_info_topic_name>camera_info</camera_info_topic_name>
-      </plugin>
-    </sensor>
-  </gazebo>
-  <!--  LIDAR  -->
-  <link name="lidar_pitch_link">
-    <visual>
-      <geometry>
-        <box size="0.04 0.04 0.01"/>
-      </geometry>
-    </visual>
-    <inertial>
-      <mass value="0.1"/>
-      <inertia ixx="0.0005" iyy="0.0005" izz="0.0005"
-              ixy="0" ixz="0" iyz="0"/>
-    </inertial>
-  </link>
-  <link name="lidar_link">
-    <visual>
-      <geometry>
-        <cylinder radius="0.015" length="0.02"/>
-      </geometry>
-    </visual>
-    <inertial>
-      <mass value="0.01"/>
-      <inertia
-        ixx="1e-5" ixy="0.0" ixz="0.0"
-        iyy="1e-5" iyz="0.0"
-        izz="1e-5"/>
-    </inertial>
-  </link>
-  <joint name="lidar_pitch_joint" type="revolute">
-    <parent link="base_link"/>
-    <child link="lidar_pitch_link"/>
-    <origin xyz="0.04 0 0.09" rpy="0 0 0"/>
-    <axis xyz="1 0 0"/>
-    <limit lower="-0.35" upper="0.35" effort="1.0" velocity="1.0"/>
-  </joint>
-  <joint name="lidar_mount_joint" type="fixed">
-    <parent link="lidar_pitch_link"/>
-    <child link="lidar_link"/>
-    <origin xyz="0 0 0.01" rpy="0 0 0"/>
-  </joint>
-  <gazebo reference="lidar_link">
-    <sensor name="lidar_sensor" type="ray">
-      <update_rate>10</update_rate>
-      <ray>
-        <scan>
-          <horizontal>
-            <samples>720</samples>
-            <min_angle>-1.5708</min_angle>
-            <max_angle>1.5708</max_angle>
-          </horizontal>
-        </scan>
-        <range>
-          <min>0.12</min>
-          <max>30.0</max>
-          <resolution>0.01</resolution>
-        </range>
-      </ray>
-      <plugin name="trip_lidar_plugin" filename="libgazebo_ros_ray_sensor.so">
-        <ros>
-          <namespace>/trip</namespace>
-          <remapping>~/out:=scan</remapping>
-        </ros>
-        <frame_name>lidar_link</frame_name>
-        <output_type>sensor_msgs/LaserScan</output_type>
-      </plugin>
-    </sensor>
-  </gazebo>
-  <xacro:macro name="wheel" params="name x y">
-    <link name="${name}">
-      <collision>
-        <geometry>
-          <cylinder radius="0.034" length="0.027"/>
-        </geometry>
-      </collision>
-      <inertial>
-        <mass value="0.1"/>
-        <inertia
-          ixx="1e-4" ixy="0" ixz="0"
-          iyy="1e-4" iyz="0"
-          izz="1e-4"/>
-      </inertial>
-    </link>
-    <joint name="${name}_joint" type="continuous">
-      <parent link="base_link"/>
-      <child link="${name}"/>
-      <origin xyz="${x} ${y} -0.042" rpy="0 ${pi/2} ${pi/2}"/>
-      <axis xyz="0 0 1"/>
-    </joint>
+  <xacro:property name='PI_2' value='1.5707963267948966'/>
+  <xacro:arg name="robot_name" default="trip" />
+  <!-- Define the macro for the whole shelfino -->
+  <xacro:macro name="trip" params='robot_name'>
+      <xacro:include filename='components/chassis.xacro' />
+      <xacro:include filename='components/lidar_scanner.xacro' />
+      <xacro:include filename='components/camera.xacro' />
+      <xacro:include filename='components/imu.xacro' />
+      <xacro:include filename='components/wheels.xacro' />
   </xacro:macro>
-  <xacro:wheel name="right_front_wheel" x="0.07"  y="-0.0716"/>
-  <xacro:wheel name="left_front_wheel"  x="0.07"  y="0.0716"/>
-  <xacro:wheel name="right_back_wheel"  x="-0.07" y="-0.0716"/>
-  <xacro:wheel name="left_back_wheel"   x="-0.07" y="0.0716"/>
+  <!-- Instantiate the model -->
+  <xacro:trip robot_name="$(arg robot_name)" />
 </robot>
