Commit message: Major changes to set up and reach first working state of gazebo

File: urdf/components/chassis.xacro (robot description, xacro)
@@ -1,4 +1,5 @@
 <?xml version="1.0"?>
 <robot name="trip" xmlns:xacro="http://www.ros.org/wiki/xacro">
+      <xacro:property name="mesh_path" value="$(env TRIP_PATH)/meshes"/>
     <material name="light_black">
         <color rgba="0.4 0.4 0.4 1.0"/>
@@ -20,5 +21,5 @@
         <origin xyz="0.003 -0.002 -0.075" rpy="0 0 ${pi}"/>
         <geometry>
-            <mesh filename="/home/davdori/trip_ws/src/TRIP-sim/trip_description/meshes/base_link.dae"/>
+            <mesh filename="${mesh_path}/base_link.dae"/>
         </geometry>
         <material name="light_black"/>

File: urdf/components/imu.xacro (robot description, xacro)
@@ -13,5 +13,5 @@
     <parent link="${robot_name}/base_link"/>
     <child link="${robot_name}/imu_link"/>
-    <origin xyz="0 0 0.08" rpy="0 0 0"/>
+    <origin xyz="0 0 0.07" rpy="0 0 0"/>
   </joint>
   <gazebo reference="${robot_name}/imu_link">

File: urdf/components/lidar_scanner.xacro (robot description, xacro)
@@ -1,9 +1,15 @@
 <?xml version="1.0"?>
 <robot name="trip" xmlns:xacro="http://www.ros.org/wiki/xacro">
+  <xacro:property name="mesh_path" value="$(env TRIP_PATH)/meshes"/>
+  <material name="blue_custom">
+      <color rgba="0.0 0.0 1.0 1.0"/>
+  </material>
   <link name="${robot_name}/lidar_pitch_link">
     <visual>
-      <geometry>
-        <box size="0.04 0.04 0.01"/>
-      </geometry>
+        <origin xyz="-0.02 0.00 0.0" rpy="0 0 ${pi}"/>
+        <geometry>
+            <mesh filename="${mesh_path}/lidar_fixed_base.dae"/>
+        </geometry>
+        <material name="blue_custom"/>
     </visual>
     <inertial>
@@ -15,7 +21,9 @@
   <link name="${robot_name}/lidar_link">
     <visual>
-      <geometry>
-        <cylinder radius="0.015" length="0.02"/>
-      </geometry>
+        <origin xyz="0.00 0.00 0.00" rpy="0 0 ${pi}"/>
+        <geometry>
+            <mesh filename="${mesh_path}/lidar.dae"/>
+        </geometry>
+        <material name="blue_custom"/>
     </visual>
     <inertial>
@@ -28,14 +36,14 @@
   </link>
   <joint name="lidar_roll_joint" type="revolute">
-    <parent link="${robot_name}/base_link"/>
-    <child link="${robot_name}/lidar_pitch_link"/>
-    <origin xyz="0.04 0 0.09" rpy="0 0 0"/>
+    <parent link="${robot_name}/lidar_pitch_link"/>
+    <child link="${robot_name}/lidar_link"/>
+    <origin xyz="0.01 0 0.01" rpy="0 0 0"/>
     <axis xyz="1 0 0"/>
     <limit lower="-0.35" upper="0.35" effort="1.0" velocity="1.0"/>
   </joint>
   <joint name="lidar_mount_joint" type="fixed">
-    <parent link="${robot_name}/lidar_pitch_link"/>
-    <child link="${robot_name}/lidar_link"/>
-    <origin xyz="0 0 0.01" rpy="0 0 0"/>
+    <parent link="${robot_name}/base_link"/>
+    <child link="${robot_name}/lidar_pitch_link"/>
+    <origin xyz="0.04 0 0.07" rpy="0 0 0"/>
   </joint>
   <gazebo reference="${robot_name}/lidar_link">
@@ -46,6 +54,6 @@
           <horizontal>
             <samples>720</samples>
-            <min_angle>-1.5708</min_angle>
-            <max_angle>1.5708</max_angle>
+            <min_angle>-3.14</min_angle>
+            <max_angle>3.14</max_angle>
           </horizontal>
         </scan>
@@ -61,5 +69,5 @@
           <remapping>~/out:=scan</remapping>
         </ros>
-        <frame_name>lidar_link</frame_name>
+        <frame_name>${robot_name}/lidar_link</frame_name>
         <output_type>sensor_msgs/LaserScan</output_type>
       </plugin>

File: urdf/components/trip.ros2_control.xacro (robot description, xacro)
@@ -57,12 +57,28 @@
     </plugin>
   </gazebo>
-  <!-- No friction for rear wheel_joints -->
+  <!-- No friction for front wheel_joints -->
+  <!-- <gazebo reference="right_front_wheel_joint">
+    <mu1 value="0.8"/>
+    <mu2 value="0.1"/>
+    <slip1>0.2</slip1>
+    <slip2>0.2</slip2>
+  </gazebo>
+  <gazebo reference="left_front_wheel_joint">
+    <mu1 value="0.8"/>
+    <mu2 value="0.1"/>
+    <slip1>0.2</slip1>
+    <slip2>0.2</slip2>
+  </gazebo>
   <gazebo reference="right_rear_wheel_joint">
-    <mu1 value="0.0"/>
-    <mu2 value="0.0"/>
+    <mu1 value="0.8"/>
+    <mu2 value="0.1"/>
+    <slip1>0.2</slip1>
+    <slip2>0.2</slip2>
   </gazebo>
   <gazebo reference="left_rear_wheel_joint">
-    <mu1 value="0.0"/>
-    <mu2 value="0.0"/>
-  </gazebo>
+    <mu1 value="0.8"/>
+    <mu2 value="0.1"/>
+    <slip1>0.2</slip1>
+    <slip2>0.2</slip2>
+  </gazebo> -->
 </robot>

File: urdf/components/wheels.xacro (robot description, xacro)
@@ -14,8 +14,9 @@
         <mass value="0.1"/>
         <inertia
-            ixx="1e-4" ixy="0" ixz="0"
-            iyy="1e-4" iyz="0"
-            izz="1e-4"/>
+            ixx="1e-3" ixy="0" ixz="0"
+            iyy="1e-3" iyz="0"
+            izz="1e-3"/>
         </inertial>
+        <mu>5.0</mu>
     </link>
     <joint name="${name}_joint" type="continuous">

File: urdf/trip.urdf.xacro (robot description, xacro)
@@ -11,4 +11,5 @@
       <xacro:include filename='components/wheels.xacro' />
       <xacro:include filename='components/trip.ros2_control.xacro' />
+      <!-- <xacro:include filename='components/gz_classic_drive.xacro' /> -->
   </xacro:macro>
   <!-- Instantiate the model -->

File: urdf/trip_rviz.urdf.xacro (robot description, xacro)
@@ -5,5 +5,5 @@
     </material>
     <!-- Base link -->
-    <link name="base_link">
+    <link name="trip/base_link">
         <inertial>
             <origin xyz="0 0 0" rpy="0 0 0"/>
@@ -15,5 +15,5 @@
         </inertial>
         <visual>
-            <origin xyz="0 0 0" rpy="0 0 3.1416"/>
+            <origin xyz="0.003 -0.002 -0.075" rpy="0 0 3.1416"/>
             <geometry>
                 <mesh filename="package://trip_description/meshes/base_link.stl" scale="1 1 1"/>
