Commit message: add parametrization of constant values for xacro

File: urdf/components/camera.xacro (robot description, xacro)
@@ -13,14 +13,14 @@
     <parent link="${robot_name}/base_link"/>
     <child link="${robot_name}/camera_link"/>
-    <origin xyz="0.08 0 0.12" rpy="0 0 0"/>
+    <origin xyz="${camera_x} ${camera_y} ${camera_z}" rpy="0 0 0"/>
   </joint>
   <gazebo reference="${robot_name}/camera_link">
     <sensor name="camera_sensor" type="camera">
-      <update_rate>30</update_rate>
+      <update_rate>${camera_fps}</update_rate>
       <camera>
-        <horizontal_fov>1.396</horizontal_fov>
+        <horizontal_fov>${camera_fov_h_rad}</horizontal_fov>
         <image>
-          <width>640</width>
-          <height>480</height>
+          <width>${camera_res_width}</width>
+          <height>${camera_res_height}</height>
           <format>R8G8B8</format>
         </image>

File: urdf/components/chassis.xacro (robot description, xacro)
@@ -1,5 +1,4 @@
 <?xml version="1.0"?>
 <robot name="trip" xmlns:xacro="http://www.ros.org/wiki/xacro">
-      <xacro:property name="mesh_path" value="$(env TRIP_PATH)/meshes"/>
     <material name="light_black">
         <color rgba="0.4 0.4 0.4 1.0"/>
@@ -12,5 +11,5 @@
     <inertial>
         <origin xyz="0 0 0" rpy="0 0 0"/>
-        <mass value="5.0"/>
+        <mass value="3.0"/>
         <inertia
         ixx="0.05" ixy="0.0" ixz="0.0"

File: urdf/components/imu.xacro (robot description, xacro)
@@ -13,5 +13,5 @@
     <parent link="${robot_name}/base_link"/>
     <child link="${robot_name}/imu_link"/>
-    <origin xyz="0 0 0.07" rpy="0 0 0"/>
+    <origin xyz="${imu_x} ${imu_y} ${imu_z}" rpy="0 0 0"/>
   </joint>
   <gazebo reference="${robot_name}/imu_link">
@@ -21,12 +21,12 @@
       <imu>
         <angular_velocity>
-          <x><noise type="gaussian"><stddev>0.002</stddev></noise></x>
-          <y><noise type="gaussian"><stddev>0.002</stddev></noise></y>
-          <z><noise type="gaussian"><stddev>0.002</stddev></noise></z>
+          <x><noise type="gaussian"><stddev>${ang_vel_noise_sigma}</stddev></noise></x>
+          <y><noise type="gaussian"><stddev>${ang_vel_noise_sigma}</stddev></noise></y>
+          <z><noise type="gaussian"><stddev>${ang_vel_noise_sigma}</stddev></noise></z>
         </angular_velocity>
         <linear_acceleration>
-          <x><noise type="gaussian"><stddev>0.03</stddev></noise></x>
-          <y><noise type="gaussian"><stddev>0.03</stddev></noise></y>
-          <z><noise type="gaussian"><stddev>0.03</stddev></noise></z>
+          <x><noise type="gaussian"><stddev>${lin_acc_noise_sigma}</stddev></noise></x>
+          <y><noise type="gaussian"><stddev>${lin_acc_noise_sigma}</stddev></noise></y>
+          <z><noise type="gaussian"><stddev>${lin_acc_noise_sigma}</stddev></noise></z>
         </linear_acceleration>
       </imu>

File: urdf/components/lidar_scanner.xacro (robot description, xacro)
@@ -1,5 +1,4 @@
 <?xml version="1.0"?>
 <robot name="trip" xmlns:xacro="http://www.ros.org/wiki/xacro">
-  <xacro:property name="mesh_path" value="$(env TRIP_PATH)/meshes"/>
   <material name="blue_custom">
       <color rgba="0.0 0.0 1.0 1.0"/>
@@ -40,10 +39,10 @@
     <origin xyz="0.01 0 0.01" rpy="0 0 0"/>
     <axis xyz="1 0 0"/>
-    <limit lower="-0.35" upper="0.35" effort="1.0" velocity="1.0"/>
+    <limit lower="${lidar_min_rot}" upper="${lidar_max_rot}" effort="1.0" velocity="1.0"/>
   </joint>
   <joint name="lidar_mount_joint" type="fixed">
     <parent link="${robot_name}/base_link"/>
     <child link="${robot_name}/lidar_pitch_link"/>
-    <origin xyz="0.04 0 0.07" rpy="0 0 0"/>
+    <origin xyz="${lidar_mount_x} ${lidar_mount_y} ${lidar_mount_z}" rpy="0 0 0"/>
   </joint>
   <gazebo reference="${robot_name}/lidar_link">
@@ -60,5 +59,5 @@
         <range>
           <min>0.12</min>
-          <max>30.0</max>
+          <max>${lidar_range}</max>
           <resolution>0.01</resolution>
         </range>

File: urdf/components/trip.ros2_control.xacro (robot description, xacro)
@@ -7,6 +7,6 @@
     <joint name="lidar_roll_joint">
       <command_interface name="position">
-          <param name="min">${-30*pi/180.0}</param>
-          <param name="max">${30*pi/180.0}</param>
+          <param name="min">${lidar_min_rot}</param>
+          <param name="max">${lidar_max_rot}</param>
       </command_interface>
       <command_interface name="velocity">
@@ -57,28 +57,3 @@
     </plugin>
   </gazebo>
-  <!-- No friction for front wheel_joints -->
-  <!-- <gazebo reference="right_front_wheel_joint">
-    <mu1 value="0.8"/>
-    <mu2 value="0.1"/>
-    <slip1>0.2</slip1>
-    <slip2>0.2</slip2>
-  </gazebo>
-  <gazebo reference="left_front_wheel_joint">
-    <mu1 value="0.8"/>
-    <mu2 value="0.1"/>
-    <slip1>0.2</slip1>
-    <slip2>0.2</slip2>
-  </gazebo>
-  <gazebo reference="right_rear_wheel_joint">
-    <mu1 value="0.8"/>
-    <mu2 value="0.1"/>
-    <slip1>0.2</slip1>
-    <slip2>0.2</slip2>
-  </gazebo>
-  <gazebo reference="left_rear_wheel_joint">
-    <mu1 value="0.8"/>
-    <mu2 value="0.1"/>
-    <slip1>0.2</slip1>
-    <slip2>0.2</slip2>
-  </gazebo> -->
 </robot>

File: urdf/components/wheels.xacro (robot description, xacro)
@@ -1,7 +1,4 @@
 <?xml version="1.0"?>
 <robot name="trip" xmlns:xacro="http://www.ros.org/wiki/xacro">
-    <xacro:property name='wheel_x_offset' value='0.07'/>
-    <xacro:property name='wheel_y_offset' value='0.0716'/>
-    <xacro:property name='wheel_radius' value='0.034'/>
     <xacro:macro name="wheel" params="name x y">
     <link name="${name}">
@@ -12,5 +9,5 @@
         </collision>
         <inertial>
-        <mass value="0.1"/>
+        <mass value="0.05"/>
         <inertia
             ixx="1e-3" ixy="0" ixz="0"
@@ -18,16 +15,16 @@
             izz="1e-3"/>
         </inertial>
-        <mu>5.0</mu>
+        <mu>${wheel_slip_mu}</mu>
     </link>
     <joint name="${name}_joint" type="continuous">
         <parent link="${robot_name}/base_link"/>
         <child link="${name}"/>
-        <origin xyz="${x} ${y} -0.042" rpy="0 ${pi/2} ${pi/2}"/>
+        <origin xyz="${x} ${y} ${wheel_z}" rpy="0 ${pi/2} ${pi/2}"/>
         <axis xyz="0 0 1"/>
     </joint>
     </xacro:macro>
-    <xacro:wheel name="right_front_wheel" x="${wheel_x_offset}"  y="${-wheel_y_offset}"/>
-    <xacro:wheel name="left_front_wheel"  x="${wheel_x_offset}"  y="${wheel_y_offset}"/>
-    <xacro:wheel name="right_rear_wheel"  x="${-wheel_x_offset}" y="${-wheel_y_offset}"/>
-    <xacro:wheel name="left_rear_wheel"   x="${-wheel_x_offset}" y="${wheel_y_offset}"/>
+    <xacro:wheel name="right_front_wheel" x="${wheel_x}"  y="${-wheel_y}"/>
+    <xacro:wheel name="left_front_wheel"  x="${wheel_x}"  y="${wheel_y}"/>
+    <xacro:wheel name="right_rear_wheel"  x="${-wheel_x}" y="${-wheel_y}"/>
+    <xacro:wheel name="left_rear_wheel"   x="${-wheel_x}" y="${wheel_y}"/>
 </robot>

File: urdf/trip.urdf.xacro (robot description, xacro)
@@ -1,8 +1,8 @@
 <?xml version="1.0"?>
 <robot name="trip" xmlns:xacro="http://www.ros.org/wiki/xacro">
-  <xacro:property name='PI_2' value='1.5707963267948966'/>
   <xacro:arg name="robot_name" default="trip" />
-  <!-- Define the macro for the whole shelfino -->
+  <!-- Define the macro for the whole robot -->
   <xacro:macro name="trip" params='robot_name'>
+      <xacro:include filename='components/constants.xacro' />
       <xacro:include filename='components/chassis.xacro' />
       <xacro:include filename='components/lidar_scanner.xacro' />
@@ -11,5 +11,4 @@
       <xacro:include filename='components/wheels.xacro' />
       <xacro:include filename='components/trip.ros2_control.xacro' />
-      <!-- <xacro:include filename='components/gz_classic_drive.xacro' /> -->
   </xacro:macro>
   <!-- Instantiate the model -->
